File: Detector_PCB_0.9/open_rad_detector.kicad_pcb (KiCad board)
At the start: 2 copper layers, 48.1 x 120.3 mm, 23 parts, among them J1 Outer_Shield, J2 Electrode, J3 Batt, J4 CONN_01X06, Q1 FMMT734, Q2 FMMT734, SW1 POWER, SW2 BUZZER, U1 LD1117S50TR, U2 MCP6N11

Commit message: Adapted to latest version of KiCad
Parts:
- RV1: footprint Potentiometers:Potentiometer_Trimmer_Piher_PT-10v10_Horizontal_Px10.0mm_Py5.0mm_MountLS -> Potentiometers:Potentiometer_Trimmer_Piher_PT-10v10_Horizontal_Px10.0mm_Py5.0mm
- U1: value LD1117S50TR -> LD1117S50TR_SOT223; footprint TO_SOT_Packages_SMD:SOT-223 -> TO_SOT_Packages_SMD:SOT-223-3_TabPin2
Connections:
- Q2 pad 1: (no net) -> Net-(Q2-Pad1)
- RV1 pad 3: (no net) -> Net-(RV1-Pad3)

Commit message: Support latest KiCad version
Connections:
- Q2 pad 1: Net-(Q2-Pad1) -> (no net)
- RV1 pad 3: Net-(RV1-Pad3) -> (no net)
Changed lines of the file:
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@@
-(kicad_pcb (version 20170123) (host pcbnew no-vcs-found-c78a2ba~59~ubuntu16.10.1)
+(kicad_pcb (version 4) (host pcbnew 4.0.7-e2-6376~58~ubuntu16.04.1)
   (general
+    (links 88)
+    (no_connects 9)
+    (area 75.997999 75.870999 124.281001 196.290001)
     (thickness 1.6)
     (drawings 8)
@@
     (zones 0)
     (modules 23)
-    (nets 17)
+    (nets 15)
   )
   (page A)
@@
       (hpglpenspeed 20)
       (hpglpendiameter 15)
+      (hpglpenoverlay 2)
       (psnegative false)
       (psa4output false)
@@
   (net 13 "Net-(D2-Pad2)")
   (net 14 "Net-(SW2-Pad3)")
-  (net 15 "Net-(Q2-Pad1)")
-  (net 16 "Net-(RV1-Pad3)")
   (net_class Default "This is the default net class."
     (clearance 0.3)
@@
     (add_net "Net-(J2-Pad1)")
     (add_net "Net-(J3-Pad2)")
-    (add_net "Net-(Q2-Pad1)")
-    (add_net "Net-(RV1-Pad3)")
     (add_net "Net-(SW2-Pad3)")
     (add_net v_comp)
@@
     (descr "module 1 pin (ou trou mecanique de percage)")
     (tags DEV)
-    (fp_text reference J2 (at -3.25628 0.04064) (layer F.SilkS)
-      (effects (font (size 1 1) (thickness 0.15)))
-    )
-    (fp_text value Electrode (at -0.254 -6.477) (layer F.Fab)
+    (fp_text reference J2 (at -3.25628 0.04064 360) (layer F.SilkS)
+      (effects (font (size 1 1) (thickness 0.15)))
+    )
+    (fp_text value Electrode (at -0.254 -6.477 360) (layer F.Fab)
       (effects (font (size 1 1) (thickness 0.15)))
     )
@@
     (tags SOT-23)
     (attr smd)
-    (fp_text reference Q1 (at -2.40284 -1.68656) (layer F.SilkS)
-      (effects (font (size 1 1) (thickness 0.15)))
-    )
-    (fp_text value FMMT734 (at 0.254 -5.334) (layer F.Fab)
-      (effects (font (size 1 1) (thickness 0.15)))
-    )
-    (fp_text user %R (at 0 0) (layer F.Fab)
+    (fp_text reference Q1 (at -2.40284 -1.68656 360) (layer F.SilkS)
+      (effects (font (size 1 1) (thickness 0.15)))
+    )
+    (fp_text value FMMT734 (at 0.254 -5.334 360) (layer F.Fab)
+      (effects (font (size 1 1) (thickness 0.15)))
+    )
+    (fp_text user %R (at 0 0 360) (layer F.Fab)
       (effects (font (size 0.5 0.5) (thickness 0.075)))
     )
@@
     (descr "Buzzer, Elektromagnetic Beeper, Summer, 12V-DC,")
     (tags "Pro Signal ABI-010-RC ")
-    (fp_text reference BZ1 (at -1.838 5.258) (layer F.SilkS)
-      (effects (font (size 1 1) (thickness 0.15)))
-    )
-    (fp_text value Buzzer (at 1.718 2.718) (layer F.Fab)
+    (fp_text reference BZ1 (at -1.838 5.258 360) (layer F.SilkS)
+      (effects (font (size 1 1) (thickness 0.15)))
+    )
+    (fp_text value Buzzer (at 1.718 2.718 360) (layer F.Fab)
       (effects (font (size 1 1) (thickness 0.15)))
     )
@@
       (effects (font (size 1 1) (thickness 0.15)))
     )
-    (fp_text user %R (at -1.838 5.258) (layer F.Fab)
+    (fp_text user %R (at -1.838 5.258 360) (layer F.Fab)
       (effects (font (size 1 1) (thickness 0.15)))
     )
@@
     (tags SOT-23)
     (attr smd)
-    (fp_text reference Q2 (at -2.3368 1.6256) (layer F.SilkS)
-      (effects (font (size 1 1) (thickness 0.15)))
-    )
-    (fp_text value FMMT734 (at 0 5.207) (layer F.Fab)
-      (effects (font (size 1 1) (thickness 0.15)))
-    )
-    (fp_text user %R (at 0 0) (layer F.Fab)
+    (fp_text reference Q2 (at -2.3368 1.6256 360) (layer F.SilkS)
+      (effects (font (size 1 1) (thickness 0.15)))
+    )
+    (fp_text value FMMT734 (at 0 5.207 360) (layer F.Fab)
+      (effects (font (size 1 1) (thickness 0.15)))
+    )
+    (fp_text user %R (at 0 0 360) (layer F.Fab)
       (effects (font (size 0.5 0.5) (thickness 0.075)))
     )
@@
     (fp_line (start 0.76 -1.58) (end -1.4 -1.58) (layer F.SilkS) (width 0.12))
     (fp_line (start 0.76 1.58) (end -0.7 1.58) (layer F.SilkS) (width 0.12))
-    (pad 1 smd rect (at -1 -0.95 270) (size 0.9 0.8) (layers F.Cu F.Paste F.Mask)
-      (net 15 "Net-(Q2-Pad1)"))
+    (pad 1 smd rect (at -1 -0.95 270) (size 0.9 0.8) (layers F.Cu F.Paste F.Mask))
     (pad 2 smd rect (at -1 0.95 270) (size 0.9 0.8) (layers F.Cu F.Paste F.Mask)
       (net 4 +BATT))
@@
     (tags "resistor 1206")
     (attr smd)
-    (fp_text reference R1 (at -1.831 -1.905) (layer F.SilkS)
-      (effects (font (size 1 1) (thickness 0.15)))
-    )
-    (fp_text value 10M (at 2.995 -0.635) (layer F.Fab)
+    (fp_text reference R1 (at -1.831 -1.905 360) (layer F.SilkS)
+      (effects (font (size 1 1) (thickness 0.15)))
+    )
+    (fp_text value 10M (at 2.995 -0.635 360) (layer F.Fab)
       (effects (font (size 1 1) (thickness 0.15)))
     )
@@
     (tags "resistor 1206")
     (attr smd)
-    (fp_text reference R2 (at 1.725 1.778) (layer F.SilkS)
-      (effects (font (size 1 1) (thickness 0.15)))
-    )
-    (fp_text value 10M (at 2.995 -0.762) (layer F.Fab)
+    (fp_text reference R2 (at 1.725 1.778 360) (layer F.SilkS)
+      (effects (font (size 1 1) (thickness 0.15)))
+    )
+    (fp_text value 10M (at 2.995 -0.762 360) (layer F.Fab)
       (effects (font (size 1 1) (thickness 0.15)))
     )
@@
     (tags "capacitor 1206")
     (attr smd)
-    (fp_text reference C3 (at 0.127 2.032) (layer F.SilkS)
-      (effects (font (size 1 1) (thickness 0.15)))
-    )
-    (fp_text value 10u (at 1.651 2.54) (layer F.Fab)
-      (effects (font (size 1 1) (thickness 0.15)))
-    )
-    (fp_text user %R (at 0.127 2.032) (layer F.Fab)
+    (fp_text reference C3 (at 0.127 2.032 360) (layer F.SilkS)
+      (effects (font (size 1 1) (thickness 0.15)))
+    )
+    (fp_text value 10u (at 1.651 2.54 360) (layer F.Fab)
+      (effects (font (size 1 1) (thickness 0.15)))
+    )
+    (fp_text user %R (at 0.127 2.032 360) (layer F.Fab)
       (effects (font (size 1 1) (thickness 0.15)))
     )
@@
     (tags "capacitor 0805")
     (attr smd)
-    (fp_text reference C4 (at -0.127 -1.905) (layer F.SilkS)
-      (effects (font (size 1 1) (thickness 0.15)))
-    )
-    (fp_text value 100n (at 1.651 -2.921) (layer F.Fab)
-      (effects (font (size 1 1) (thickness 0.15)))
-    )
-    (fp_text user %R (at -0.127 -1.905) (layer F.Fab)
+    (fp_text reference C4 (at -0.127 -1.905 360) (layer F.SilkS)
+      (effects (font (size 1 1) (thickness 0.15)))
+    )
+    (fp_text value 100n (at 1.651 -2.921 360) (layer F.Fab)
+      (effects (font (size 1 1) (thickness 0.15)))
+    )
+    (fp_text user %R (at -0.127 -1.905 360) (layer F.Fab)
       (effects (font (size 1 1) (thickness 0.15)))
     )
@@
   (module SW_JS202011SCQN:SW_JS202011SCQN (layer F.Cu)
     (at 89 158 270)
-    (fp_text reference SW1 (at 5.068 0) (layer F.SilkS)
-      (effects (font (size 1 1) (thickness 0.15)))
-    )
-    (fp_text value POWER (at -0.266 6.958) (layer F.SilkS)
+    (fp_text reference SW1 (at 5.068 0 360) (layer F.SilkS)
+      (effects (font (size 1 1) (thickness 0.15)))
+    )
+    (fp_text value POWER (at -0.266 6.958 360) (layer F.SilkS)
       (effects (font (size 1 1) (thickness 0.15)))
     )
@@
     (tags "resistor 0805")
     (attr smd)
-    (fp_text reference R3 (at -2.032 0.127) (layer F.SilkS)
-      (effects (font (size 1 1) (thickness 0.15)))
-    )
-    (fp_text value R_G (at 0 2.413) (layer F.Fab)
+    (fp_text reference R3 (at -2.032 0.127 360) (layer F.SilkS)
+      (effects (font (size 1 1) (thickness 0.15)))
+    )
+    (fp_text value R_G (at 0 2.413 360) (layer F.Fab)
       (effects (font (size 1 1) (thickness 0.15)))
     )
@@
     (tags "Diode 1206")
     (attr smd)
-    (fp_text reference D2 (at 0.024 -2.286) (layer F.SilkS)
-      (effects (font (size 1 1) (thickness 0.15)))
-    )
-    (fp_text value D (at 0.024 1.9) (layer F.Fab)
-      (effects (font (size 1 1) (thickness 0.15)))
-    )
-    (fp_text user %R (at 0 -2.286) (layer F.Fab)
+    (fp_text reference D2 (at 0.024 -2.286 360) (layer F.SilkS)
+      (effects (font (size 1 1) (thickness 0.15)))
+    )
+    (fp_text value D (at 0.024 1.9 360) (layer F.Fab)
+      (effects (font (size 1 1) (thickness 0.15)))
+    )
+    (fp_text user %R (at 0 -2.286 360) (layer F.Fab)
       (effects (font (size 1 1) (thickness 0.15)))
     )
@@
   (module SW_JS202011SCQN:SW_JS202011SCQN (layer F.Cu)
     (at 111 158 270)
-    (fp_text reference SW2 (at 5.068 0) (layer F.SilkS)
-      (effects (font (size 1 1) (thickness 0.15)))
-    )
-    (fp_text value BUZZER (at -0.266 -7.364) (layer F.SilkS)
+    (fp_text reference SW2 (at 5.068 0 360) (layer F.SilkS)
+      (effects (font (size 1 1) (thickness 0.15)))
+    )
+    (fp_text value BUZZER (at -0.266 -7.364 360) (layer F.SilkS)
       (effects (font (size 1 1) (thickness 0.15)))
     )
@@
     (tags "resistor 1206")
     (attr smd)
-    (fp_text reference R5 (at -2.71492 0.34544) (layer F.SilkS)
-      (effects (font (size 1 1) (thickness 0.15)))
-    )
-    (fp_text value 10M (at 2.98992 0.7112) (layer F.Fab)
+    (fp_text reference R5 (at -2.71492 0.34544 360) (layer F.SilkS)
+      (effects (font (size 1 1) (thickness 0.15)))
+    )
+    (fp_text value 10M (at 2.98992 0.7112 360) (layer F.Fab)
       (effects (font (size 1 1) (thickness 0.15)))
     )
@@
     (pad 2 thru_hole circle (at 10 -2.5 90) (size 2.34 2.34) (drill 1.3) (layers *.Cu *.Mask)
       (net 8 v_out))
-    (pad 3 thru_hole circle (at 0 -5 90) (size 2.34 2.34) (drill 1.3) (layers *.Cu *.Mask)
-      (net 16 "Net-(RV1-Pad3)"))
+    (pad 3 thru_hole circle (at 0 -5 90) (size 2.34 2.34) (drill 1.3) (layers *.Cu *.Mask))
     (model Potentiometers.3dshapes/Potentiometer_Trimmer_Piher_PT-10v10_Horizontal_Px10.0mm_Py5.0mm.wrl
       (at (xyz 0 0 0))
